File: AmpliAudio/AmpliAudio.kicad_pcb (KiCad board)
At the start: 2 copper layers, 110 x 100 mm, 52 parts, among them J2 Conn_01x02, J3 Conn_01x03, Q1 2N2907, Q10 TIP32, Q11 BD138, Q12 TIP31, Q13 2N2222, Q2 2N2907, Q3 2N2907, Q4 2N2222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

Commit message: avis placement
Parts:
- moved U1 84.7 mm to (58.0, 71.0), turned to 0 degrees
- moved Dz1 82.5 mm to (34.0, 107.0), turned to 270 degrees
- moved C7 78.5 mm to (134.0, 96.0)
- moved RV2 78.0 mm to (62.0, 96.0)
- moved R5 61.4 mm to (40.0, 120.8), turned to 270 degrees
- moved Q8 60.3 mm to (82.0, 89.0)
- moved C4 59.0 mm to (129.0, 84.0)
- moved R12 58.1 mm to (94.0, 67.0), turned to 0 degrees
- moved R1 56.0 mm to (53.0, 137.0), turned to 270 degrees
- moved C11 54.6 mm to (122.0, 58.0), turned to 0 degrees
- moved R13 52.4 mm to (75.0, 62.0)
- moved R11 48.4 mm to (57.0, 67.0), turned to 0 degrees
- moved R3 47.8 mm to (46.0, 120.8), turned to 270 degrees
- moved C10 47.5 mm to (133.0, 69.0)
- moved R4 47.4 mm to (67.0, 131.0)
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
Commit message: Avis routage
Parts:
- moved R14 56.3 mm to (54.0, 131.0)
- moved R15 56.3 mm to (59.7, 120.8)
- moved D1 14.1 mm to (132.0, 131.0), turned to 90 degrees
- moved R9 13.0 mm to (86.0, 130.7)
- moved D2 10.0 mm to (117.0, 114.0), turned to 90 degrees
- moved J3 9.37 mm to (67.0, 60.6), turned to 180 degrees
- moved U2 6.50 mm to (59.0, 150.0)
- moved C4 6.32 mm to (135.0, 86.0), turned to 180 degrees
- moved J2 6.08 mm to (112.5, 60.6), turned to 180 degrees
- moved Q4 6.00 mm to (92.9, 129.2)
- moved Q5 6.00 mm to (106.0, 129.0)
- moved Q6 6.00 mm to (105.0, 115.0)
- moved Q7 6.00 mm to (93.3, 115.4)
- moved C9 5.87 mm to (49.0, 61.3), turned to 180 degrees
- moved R13 5.83 mm to (78.0, 67.0)
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Connections:
- J2 pad 1: Net-(J2-Pad1) -> GND
- J2 pad 2: GND -> Net-(J2-Pad2)
- R8 pad 2: Net-(C2-Pad1) -> Net-(R8-Pad2)
- RV1 pad 3: Net-(C2-Pad1) -> Net-(R8-Pad2)
- U1 pad c2: Net-(J2-Pad1) -> Net-(J2-Pad2)
Routing:
- net Net-(C2-Pad1): track 0.00 -> 787.6 mm
- net Net-(Q6-Pad3): track 0.00 -> 417.9 mm
- net GND: track 0.00 -> 405.2 mm
- net +12V: track 0.00 -> 371.1 mm
- net -12V: track 0.00 -> 313.9 mm
- net Net-(R11-Pad2): track 0.00 -> 244.8 mm
- net Net-(Q6-Pad2): track 0.00 -> 214.8 mm
- net Net-(C2-Pad2): track 0.00 -> 157.4 mm
- net Net-(D1-Pad2): track 0.00 -> 153.5 mm
- net Net-(Q11-Pad1): track 0.00 -> 124.2 mm
- net Net-(Q6-Pad1): track 0.00 -> 100.8 mm
- net Net-(C1-Pad1): track 0.00 -> 70.3 mm
- net Net-(Q4-Pad1): track 0.00 -> 30.4 mm
- net Net-(Q2-Pad2): track 0.00 -> 29.1 mm
- net Net-(Q3-Pad1): track 0.00 -> 28.0 mm
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- added copper zone on B.Cu, net GND
Other:
- board text added: "Paul NOUGUE & Alassane GUEYE 3IMACS D - Projet Ampli Audio INSA"

Commit message: Version Finale
Connections:
- Q9 pad 1: Net-(Q10-Pad1) -> Net-(Q10-Pad2)
- Q9 pad 2: Net-(Q10-Pad2) -> Net-(Q10-Pad1)
Routing:
- net Net-(Q11-Pad1): track 124.2 -> 40.7 mm
- net Net-(Q10-Pad1): track 5.00 -> 15.0 mm
- net -12V: track 313.9 -> 323.0 mm
- net Net-(D1-Pad2): track 153.5 -> 150.2 mm
- net Net-(C2-Pad1): track 787.6 -> 784.5 mm
- net Net-(Q10-Pad2): track 23.1 -> 25.1 mm
- net GND: track 405.2 -> 403.5 mm
- net Net-(R11-Pad2): track 244.8 -> 243.3 mm
- net Net-(Q6-Pad3): track 417.9 -> 418.9 mm
