File: AmpliAudio/AmpliAudio.sch (KiCad schematic (older format))
At the start: 52 parts, among them J2 Conn_01x02, J3 Conn_01x03, Q1 2N2907, Q10 TIP32, Q11 BD138, Q12 TIP31, Q13 2N2222, Q2 2N2907, Q3 2N2907, Q4 2N2222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

Commit message: Avis routage
Connections:
- net GND: now also J2.1 (Pin_1); no longer J2.2 (Pin_2)
- net at C2.1, Q11.3 (B), Q4.3 (C)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: no longer R8.2, RV1.3
- net at U1.c2: now also J2.2 (Pin_2); no longer J2.1 (Pin_1)
- new net: R8.2, RV1.3
Changed lines of the file:
@@
 Sheet 1 1
 Title "Projet Ampli"
-Date "2020-03-23"
+Date "2020-04-15"
 Rev ""
 Comp "Paul NOUGUE-Alassane GUEYE"
@@
 Wire Wire Line
 	5450 2750 5350 2750
-Connection ~ 5350 2750
-Wire Wire Line
-	5350 2750 5350 3500
 $Comp
 L Device:R R15
@@
 L Connector_Generic:Conn_01x02 J2
 U 1 1 5E67BFD2
-P 10700 2550
-F 0 "J2" H 10780 2542 50  0000 L CNN
-F 1 "Conn_01x02" H 10780 2451 50  0000 L CNN
-F 2 "CmpAmpliAudio:PhoenixContact_MSTBVA_2,5_2-G-5,08_1x02_P5.08mm_Vertical" H 10700 2550 50  0001 C CNN
-F 3 "~" H 10700 2550 50  0001 C CNN
-	1    10700 2550
-	1    0    0    -1
-$EndComp
-Wire Wire Line
+P 10700 2650
+F 0 "J2" H 10780 2642 50  0000 L CNN
+F 1 "Conn_01x02" H 10780 2551 50  0000 L CNN
+F 2 "CmpAmpliAudio:PhoenixContact_MSTBVA_2,5_2-G-5,08_1x02_P5.08mm_Vertical" H 10700 2650 50  0001 C CNN
+F 3 "~" H 10700 2650 50  0001 C CNN
+	1    10700 2650
+	1    0    0    1
+$EndComp
+Wire Wire Line

Commit message: Version Finale
Parts:
- removed Q9: BD139, CmpAmpliAudio:TO-126-3_Vertical, symbol Device:Q_NPN_CEB
- added Q9: BD139, CmpAmpliAudio:TO-126-3_Vertical, symbol Device:Q_NPN_ECB
Connections:
- net at Q6.3 (C), Q8.2 (C), RV1.1: now also Q9.3 (B)
- net at Q10.1 (B): now also Q9.2 (C)
- net at Q10.2 (C), R11.1: now also Q9.1 (E)
Changed lines of the file:
@@
 	7050 3000 7050 2950
-$Comp
-L Device:Q_NPN_CEB Q9
-U 1 1 5E6AC056
-P 6500 1850
-F 0 "Q9" H 6691 1896 50  0000 L CNN
-F 1 "BD139" H 6691 1805 50  0000 L CNN
-F 2 "CmpAmpliAudio:TO-126-3_Vertical" H 6700 1950 50  0001 C CNN
-F 3 "~" H 6500 1850 50  0001 C CNN
-	1    6500 1850
-	1    0    0    -1
-$EndComp
 $Comp
 L Device:Q_PNP_ECB Q11
@@
 Wire Wire Line
 	2000 3300 1950 3300
+$Comp
+L Device:Q_NPN_ECB Q9
+U 1 1 5E9A541F
+P 6500 1850
+F 0 "Q9" H 6691 1896 50  0000 L CNN
+F 1 "BD139" H 6691 1805 50  0000 L CNN
+F 2 "CmpAmpliAudio:TO-126-3_Vertical" H 6700 1950 50  0001 C CNN
+F 3 "~" H 6500 1850 50  0001 C CNN
+	1    6500 1850
+	1    0    0    -1
+$EndComp
 $EndSCHEMATC
